Commit message: sepearate ros2_control.xacro

File: kortex_moveit_config/kinova_gen3_lite_moveit_config/config/gen3_lite.ros2_control.xacro (robot description, xacro)
@@ -50,11 +50,4 @@
                 <state_interface name="velocity"/>
             </joint>
-            <joint name="right_finger_bottom_joint">
-                <command_interface name="position"/>
-                <state_interface name="position">
-                  <param name="initial_value">${initial_positions['right_finger_bottom_joint']}</param>
-                </state_interface>
-                <state_interface name="velocity"/>
-            </joint>
         </ros2_control>
     </xacro:macro>

File: kortex_moveit_config/kinova_gen3_lite_moveit_config/config/gen3_lite.urdf.xacro (robot description, xacro)
@@ -6,4 +6,6 @@
     <!-- Import control_xacro -->
     <xacro:include filename="gen3_lite.ros2_control.xacro" />
+    <xacro:include filename="gen3_lite_hand.ros2_control.xacro" />
     <xacro:gen3_lite_ros2_control name="FakeSystem" initial_positions_file="$(arg initial_positions_file)"/>
+    <xacro:gen3_lite_hand_ros2_control name="FakeHandSystem" initial_positions_file="$(arg initial_positions_file)"/>
 </robot>

Commit message: hem

File: kortex_moveit_config/kinova_gen3_lite_moveit_config/config/gen3_lite.ros2_control.xacro (robot description, xacro)
@@ -50,11 +50,4 @@
                 <state_interface name="velocity"/>
             </joint>
-            <joint name="right_finger_bottom_joint">
-                <command_interface name="position"/>
-                <state_interface name="position">
-                  <param name="initial_value">${initial_positions['right_finger_bottom_joint']}</param>
-                </state_interface>
-                <state_interface name="velocity"/>
-            </joint>
         </ros2_control>
     </xacro:macro>

File: kortex_moveit_config/kinova_gen3_lite_moveit_config/config/gen3_lite.urdf.xacro (robot description, xacro)
@@ -6,4 +6,7 @@
     <!-- Import control_xacro -->
     <xacro:include filename="gen3_lite.ros2_control.xacro" />
+    <xacro:include filename="gen3_lite_hand.ros2_control.xacro" />
     <xacro:gen3_lite_ros2_control name="FakeSystem" initial_positions_file="$(arg initial_positions_file)"/>
+    <xacro:gen3_lite_hand_ros2_control name="HandFakeSystem"/>
+    <!-- <xacro:gen3_lite_ros2_control name="FakeSystem" initial_positions_file="$(arg initial_positions_file)" ros2_control_hardware_type="$(arg ros2_control_hardware_type)"/> -->
 </robot>

Commit message: pick@place plan & exec success

File: kortex_moveit_config/kinova_gen3_lite_moveit_config/config/gen3_lite.ros2_control.xacro (robot description, xacro)
@@ -1,10 +1,16 @@
 <?xml version="1.0"?>
 <robot xmlns:xacro="http://www.ros.org/wiki/xacro">
-    <xacro:macro name="gen3_lite_ros2_control" params="name initial_positions_file">
+    <xacro:macro name="gen3_lite_ros2_control" params="name initial_positions_file ros2_control_hardware_type">
         <xacro:property name="initial_positions" value="${load_yaml(initial_positions_file)['initial_positions']}"/>
         <ros2_control name="${name}" type="system">
             <hardware>
-                <!-- By default, set up controllers for simulation. This won't work on real hardware -->
-                <plugin>mock_components/GenericSystem</plugin>
+                <xacro:if value="${ros2_control_hardware_type == 'mock_components'}">
+                    <plugin>mock_components/GenericSystem</plugin>
+                </xacro:if>
+                <xacro:if value="${ros2_control_hardware_type == 'isaac'}">
+                    <plugin>topic_based_ros2_control/TopicBasedSystem</plugin>
+                    <param name="joint_commands_topic">/isaac_joint_commands</param>
+                    <param name="joint_states_topic">/isaac_joint_states</param>
+                </xacro:if>
             </hardware>
             <joint name="joint_1">

File: kortex_moveit_config/kinova_gen3_lite_moveit_config/config/gen3_lite.urdf.xacro (robot description, xacro)
@@ -2,4 +2,5 @@
 <robot xmlns:xacro="http://www.ros.org/wiki/xacro" name="gen3_lite">
     <xacro:arg name="initial_positions_file" default="initial_positions.yaml" />
+    <xacro:arg name="ros2_control_hardware_type" default="mock_components" />
     <!-- Import gen3_lite urdf file -->
     <xacro:include filename="$(find kortex_description)/robots/gen3_lite.urdf" />
@@ -7,6 +8,8 @@
     <xacro:include filename="gen3_lite.ros2_control.xacro" />
     <xacro:include filename="gen3_lite_hand.ros2_control.xacro" />
-    <xacro:gen3_lite_ros2_control name="FakeSystem" initial_positions_file="$(arg initial_positions_file)"/>
-    <xacro:gen3_lite_hand_ros2_control name="HandFakeSystem"/>
+    <xacro:gen3_lite_ros2_control name="FakeSystem" initial_positions_file="$(arg initial_positions_file)" ros2_control_hardware_type="$(arg ros2_control_hardware_type)"/>
+    <xacro:gen3_lite_hand_ros2_control name="HandFakeSystem" initial_positions_file="$(arg initial_positions_file)" ros2_control_hardware_type="$(arg ros2_control_hardware_type)"/>
+    <!-- <xacro:gen3_lite_ros2_control name="FakeSystem" initial_positions_file="$(arg initial_positions_file)"/>
+    <xacro:gen3_lite_hand_ros2_control name="HandFakeSystem"/> -->
     <!-- <xacro:gen3_lite_ros2_control name="FakeSystem" initial_positions_file="$(arg initial_positions_file)" ros2_control_hardware_type="$(arg ros2_control_hardware_type)"/> -->
 </robot>

File: kortex_moveit_config/kinova_gen3_lite_moveit_config/config/gen3_lite_hand.ros2_control.xacro (robot description, xacro)
@@ -1,9 +1,16 @@
 <?xml version="1.0"?>
 <robot xmlns:xacro="http://www.ros.org/wiki/xacro">
-    <xacro:macro name="gen3_lite_hand_ros2_control" params="name ros2_control_hardware_type">
+    <xacro:macro name="gen3_lite_hand_ros2_control" params="name initial_positions_file ros2_control_hardware_type">
+        <xacro:property name="initial_positions" value="${load_yaml(initial_positions_file)['initial_positions']}"/>
         <ros2_control name="${name}" type="system">
             <hardware>
-                <!-- By default, set up controllers for simulation. This won't work on real hardware -->
-                <plugin>mock_components/GenericSystem</plugin>
+                <xacro:if value="${ros2_control_hardware_type == 'mock_components'}">
+                    <plugin>mock_components/GenericSystem</plugin>
+                </xacro:if>
+                <xacro:if value="${ros2_control_hardware_type == 'isaac'}">
+                    <plugin>topic_based_ros2_control/TopicBasedSystem</plugin>
+                    <param name="joint_commands_topic">/isaac_joint_commands</param>
+                    <param name="joint_states_topic">/isaac_joint_states</param>
+                </xacro:if>
             </hardware>
             <joint name="right_finger_bottom_joint">
@@ -14,4 +21,25 @@
                 <state_interface name="velocity"/>
             </joint>
+            <!-- <joint name="left_finger_bottom_joint">
+                <command_interface name="position"/>
+                <state_interface name="position">
+                  <param name="initial_value">${initial_positions['right_finger_bottom_joint']}</param>
+                </state_interface>
+                <state_interface name="velocity"/>
+            </joint>
+            <joint name="left_finger_tip_joint">
+                <command_interface name="position"/>
+                <state_interface name="position">
+                  <param name="initial_value">${initial_positions['right_finger_bottom_joint']}</param>
+                </state_interface>
+                <state_interface name="velocity"/>
+            </joint>
+            <joint name="right_finger_tip_joint">
+                <command_interface name="position"/>
+                <state_interface name="position">
+                  <param name="initial_value">${initial_positions['right_finger_bottom_joint']}</param>
+                </state_interface>
+                <state_interface name="velocity"/>
+            </joint> -->
         </ros2_control>
     </xacro:macro>
