Commit message: changed to eef_name hand

File: kortex_moveit_config/kinova_gen3_lite_moveit_config/config/gen3_lite_hand.ros2_control.xacro (robot description, xacro)
@@ -1,5 +1,5 @@
 <?xml version="1.0"?>
 <robot xmlns:xacro="http://www.ros.org/wiki/xacro">
-    <xacro:macro name="gen3_lite_ros2_control" params="name initial_positions_file">
+    <xacro:macro name="gen3_lite_hand_ros2_control" params="name initial_positions_file">
         <xacro:property name="initial_positions" value="${load_yaml(initial_positions_file)['initial_positions']}"/>
         <ros2_control name="${name}" type="system">

Commit message: why

File: kortex_moveit_config/kinova_gen3_lite_moveit_config/config/gen3_lite_hand.ros2_control.xacro (robot description, xacro)
@@ -21,5 +21,5 @@
                 <state_interface name="velocity"/>
             </joint>
-            <!-- <joint name="left_finger_bottom_joint">
+            <joint name="left_finger_bottom_joint">
                 <command_interface name="position"/>
                 <state_interface name="position">
@@ -41,5 +41,5 @@
                 </state_interface>
                 <state_interface name="velocity"/>
-            </joint> -->
+            </joint>
         </ros2_control>
     </xacro:macro>
